Commit message: feat: add set_zero command support, update joint limits, and improve rclpy shutdown handling

File: src/eb15_description/urdf/eb15.urdf (robot description, URDF)
Before this commit: robot eb15, 6 links, 5 joints
Joints:
- joint joint2: limit lower=-3.14159 upper=3.14159 effort=15.0 velocity=3.14 -> lower=-1.570796 upper=1.570796 effort=15.0 velocity=3.14

Commit message: feat: add wrist and gripper CAD meshes and update robot description and driver configuration

File: src/eb15_description/urdf/eb15.urdf (robot description, URDF)
Before this commit: robot eb15, 6 links, 5 joints
Links:
- added link wrist_base_link, mass 0.08; collision cylinder length=0.026 radius=0.028; visual mesh filename=package://eb15_description/meshes/wrist_base.stl scale=0.001 0.001 0.001
- added link wrist_link, mass 0.22; collision box size=0.082 0.069 0.075; visual mesh filename=package://eb15_description/meshes/wrist_rot.stl scale=0.001 0.001 0.001
- link tool0: geometry visual cylinder length=0.004 radius=0.025
Joints:
- added joint wrist_base_joint: type fixed, parent link3, child wrist_base_link, origin xyz=0 0 0.178 rpy=0 0 0
- added joint wrist_joint: type revolute, parent wrist_base_link, child wrist_link, origin xyz=0 0 0 rpy=0 0 0, axis 0 0 1, limit lower=-1.570796 upper=1.570796 effort=5.0 velocity=3.14
- joint tool_joint: origin xyz=0 0 0.178 rpy=0 0 0 -> xyz=0 0 0.0717 rpy=0 0 0; parent link3 -> wrist_link

Commit message: feat: add EBG-20 adaptive robot gripper model and update joint configurations in URDF and driver

File: src/eb15_description/urdf/eb15.urdf (robot description, URDF)
Before this commit: robot eb15, 8 links, 7 joints
Links:
- added link gripper_base_link, mass 0.22; collision box size=0.085 0.065 0.077; visual mesh filename=package://eb15_description/meshes/gripper_base.stl scale=0.001 0.001 0.001
- added link gripper_left_finger_link, mass 0.04; collision box size=0.015 0.021 0.040; visual mesh filename=package://eb15_description/meshes/gripper_left_finger.stl scale=0.001 0.001 0.001
- added link gripper_right_finger_link, mass 0.04; collision box size=0.015 0.021 0.040; visual mesh filename=package://eb15_description/meshes/gripper_right_finger.stl scale=0.001 0.001 0.001
- added link gripper_tcp; visual sphere radius=0.004
- link tool0: geometry 
- link wrist_base_link: mass 0.08 -> 0.22; geometry collision box size=0.082 0.069 0.075; visual mesh filename=package://eb15_description/meshes/wrist_base.stl scale=0.001 0.001 0.001
- link wrist_link: mass 0.22 -> 0.08; geometry collision cylinder length=0.029 radius=0.028; visual mesh filename=package://eb15_description/meshes/wrist_rot.stl scale=0.001 0.001 0.001
Joints:
- added joint gripper_base_joint: type fixed, parent tool0, child gripper_base_link, origin xyz=0 0 0 rpy=0 0 0
- added joint gripper_left_joint: type prismatic, parent gripper_base_link, child gripper_left_finger_link, origin xyz=0 0 0 rpy=0 0 0, axis 1 0 0, limit lower=0.0 upper=0.020 effort=20.0 velocity=0.05
- added joint gripper_right_joint: type prismatic, parent gripper_base_link, child gripper_right_finger_link, origin xyz=0 0 0 rpy=0 0 0, axis -1 0 0, limit lower=0.0 upper=0.020 effort=20.0 velocity=0.05, mimic joint=gripper_left_joint multiplier=1.0 offset=0.0
- added joint gripper_tcp_joint: type fixed, parent gripper_base_link, child gripper_tcp, origin xyz=0 0 0.098 rpy=0 0 0
- joint tool_joint: origin xyz=0 0 0.0717 rpy=0 0 0 -> xyz=0 0 0.0877 rpy=0 0 0

Commit message: feat:Robot Gripper URDF updated

File: src/eb15_description/urdf/eb15.urdf (robot description, URDF)
Before this commit: robot eb15, 12 links, 11 joints
Joints:
- joint gripper_base_joint: origin xyz=0 0 0 rpy=0 0 0 -> xyz=0 0 -0.0095 rpy=0 0 0

Commit message: feat: add elbow limit switches, homing routines, and update joint limits in URDF and driver

File: src/eb15_description/urdf/eb15.urdf (robot description, URDF)
Before this commit: robot eb15, 12 links, 11 joints
Joints:
- joint gripper_left_joint: limit lower=0.0 upper=0.020 effort=20.0 velocity=0.05 -> lower=-0.016 upper=0.012 effort=20.0 velocity=0.05
- joint gripper_right_joint: limit lower=0.0 upper=0.020 effort=20.0 velocity=0.05 -> lower=-0.016 upper=0.012 effort=20.0 velocity=0.05
- joint joint3: limit lower=-3.14159 upper=3.14159 effort=12.0 velocity=3.14 -> lower=-2.700 upper=2.700 effort=12.0 velocity=3.14

Commit message: feat: modularize robot description into xacro components and add joint limits configuration

File: src/eb15_description/urdf/eb15.urdf (robot description, URDF)
Before this commit: robot eb15, 12 links, 11 joints
Joints:
- joint joint3: limit lower=-2.700 upper=2.700 effort=12.0 velocity=3.14 -> lower=-2.7 upper=2.7 effort=12.0 velocity=3.14

Commit message: refactor: rotate wrist_base_joint -90 degrees to align servo axis with elbow axis

File: src/eb15_description/urdf/eb15.urdf (robot description, URDF)
Before this commit: robot eb15, 12 links, 11 joints
Joints:
- joint wrist_base_joint: origin xyz=0 0 0.178 rpy=0 0 0 -> xyz=0 0 0.178 rpy=0 0 -1.5707963

File: src/eb15_description/urdf/forearm.xacro (robot description, xacro)
@@ -60,5 +60,6 @@
     <parent link="link3"/>
     <child link="wrist_base_link"/>
-    <origin xyz="0 0 0.178" rpy="0 0 0"/>
+    <!-- Rotated -90 deg (-pi/2 rad) clockwise so servo axis aligns with elbow axis -->
+    <origin xyz="0 0 0.178" rpy="0 0 -1.5707963"/>
   </joint>
   <link name="wrist_base_link">

Commit message: fix: resolve MoveIt start-state bounds errors by padding gripper limits and removing mimic joints from SRDF

File: src/eb15_description/urdf/eb15.urdf (robot description, URDF)
Before this commit: robot eb15, 12 links, 11 joints
Joints:
- joint gripper_left_joint: limit lower=-0.016 upper=0.012 effort=20.0 velocity=0.05 -> lower=-0.018 upper=0.015 effort=20.0 velocity=0.05
- joint gripper_right_joint: limit lower=-0.016 upper=0.012 effort=20.0 velocity=0.05 -> lower=-0.018 upper=0.015 effort=20.0 velocity=0.05

File: src/eb15_description/urdf/gripper.xacro (robot description, xacro)
@@ -1,7 +1,7 @@
 <?xml version="1.0"?>
 <robot xmlns:xacro="http://www.ros.org/wiki/xacro">
-  <!-- Gripper Stroke Limits -->
-  <xacro:property name="gripper_open_limit"  value="-0.016"/>
-  <xacro:property name="gripper_close_limit" value="0.012"/>
+  <!-- Gripper Stroke Limits (padded bounds to prevent float32/float64 edge violations in MoveIt) -->
+  <xacro:property name="gripper_open_limit"  value="-0.018"/>
+  <xacro:property name="gripper_close_limit" value="0.015"/>
   <!-- ================================================= -->
   <!-- EBG-20 ADAPTIVE ROBOT GRIPPER                     -->
